Commit message: Updated markers and aruco launching

File: cp3_base/robot_description/cp3/urdf/turtlebot_properties.urdf.xacro (robot description, xacro)
@@ -19,5 +19,5 @@
      (currently in development and awaiting feedback)
    -->
-	<xacro:property name="cam_px" value="0.15" />
+	<xacro:property name="cam_px" value="0.25" />
 <!--	<xacro:property name="cam_py" value="-0.0125" /> Y varies for different configurations. get sets in sensors_urdf -->
 	<xacro:property name="cam_pz" value="0.2870" />
