Commit message: This is really a stash, but there are a lot of temporary files

File: cp3_base/robot_description/cp3/urdf/hokuyo.urdf.xacro (robot description, xacro)
@@ -5,5 +5,5 @@
   <xacro:macro name="sensor_hokuyo" params="parent">
     <joint name="laser" type="fixed">
-      <origin xyz="0.15 0.0 1.5" rpy="3.14159 0.0 0.0" />
+      <origin xyz="0.1 0.0 0.425" rpy="3.14159 0.0 0.0" />
       <parent link="base_link" />
       <child link="base_laser_link" />
@@ -12,5 +12,5 @@
       <visual>
         <geometry>
-          <mesh filename="package://turtlebot_description/meshes/sensors/hokuyo.dae"/>
+          <mesh filename="package://cp3_base/robot_description/cp3/meshes/hokuyo.dae"/>
         </geometry>
       </visual>

File: cp3_base/robot_description/cp3/urdf/kobuki_hexagons_kinect.urdf.xacro (robot description, xacro)
@@ -6,5 +6,5 @@
 -->
 <robot name="turtlebot" xmlns:xacro="http://ros.org/wiki/xacro">
-  <xacro:include filename="$(find turtlebot_description)/urdf/turtlebot_common_library.urdf.xacro" />
+  <xacro:include filename="$(find cp3_base)/robot_description/cp3/urdf/turtlebot_common_library.urdf.xacro" />
   <xacro:include filename="$(find kobuki_description)/urdf/kobuki.urdf.xacro" />
   <xacro:include filename="$(find turtlebot_description)/urdf/stacks/hexagons.urdf.xacro"/>
@@ -14,6 +14,8 @@
   <xacro:include filename="$(find cp3_base)/robot_description/cp3/urdf/kinect.urdf.xacro"/>
   <xacro:include filename="$(find cp3_base)/robot_description/cp3/urdf/hokuyo.urdf.xacro"/>
+  <xacro:include filename="$(find cp3_base)/robot_description/cp3/urdf/camera360.urdf.xacro"/>
   <kobuki/>
   <stack_hexagons parent="base_link"/>
+  <sensor_camera360 parent="base_link"/>
   <sensor_kinect  parent="base_link"/>
   <sensor_hokuyo  parent="base_link"/>

File: cp3_base/robot_description/cp3/urdf/turtlebot_common_library.urdf.xacro (robot description, xacro)
@@ -6,4 +6,4 @@
   <!-- General -->
   <xacro:include filename="$(find turtlebot_description)/urdf/common_properties.urdf.xacro"/>
-  <xacro:include filename="$(find turtlebot_description)/urdf/turtlebot_properties.urdf.xacro"/>
+  <xacro:include filename="$(find cp3_base)/robot_description/cp3/urdf/turtlebot_properties.urdf.xacro"/>
 </robot>

File: cp3_base/robot_description/cp3/urdf/turtlebot_gazebo.urdf.xacro (robot description, xacro)
@@ -8,5 +8,5 @@
         <update_rate>20.0</update_rate>
         <camera>
-          <horizontal_fov>${120.0*M_PI/180.0}</horizontal_fov>
+          <horizontal_fov>${140.0*M_PI/180.0}</horizontal_fov>
           <image>
             <format>B8G8R8</format>
@@ -76,3 +76,36 @@
     </gazebo>
   </xacro:macro>
+  <xacro:macro name="camera360">
+    <gazebo reference="camera360_link">
+      <sensor type="camera" name="camera360">
+        <update_rate>30.0</update_rate>
+        <camera name="camera360">
+          <horizontal_fov>${140.0*M_PI/180.0}</horizontal_fov>
+          <image>
+            <format>B8G8R8</format>
+            <width>1280</width> <!-- 3840 -->
+            <height>480</height>
+          </image>
+          <clip>
+            <near>0.05</near>
+            <far>8.0</far>
+          </clip>
+        </camera>
+        <plugin name="camera_controller" filename="libgazebo_ros_camera.so">
+          <alwaysOn>true</alwaysOn>
+          <updateRate>10.0</updateRate>
+          <cameraName>camera360</cameraName>
+          <imageTopicName>image_raw</imageTopicName>
+          <cameraInfoTopicName>camera_info</cameraInfoTopicName>
+          <frameName>camera360_link</frameName>
+          <hackBaseline>0.1</hackBaseline>
+          <distortion_k1>0.0</distortion_k1>
+          <distortion_k2>0.0</distortion_k2>
+          <distortion_k3>0.0</distortion_k3>
+          <distortion_t1>0.0</distortion_t1>
+          <distortion_t2>0.0</distortion_t2>
+        </plugin>
+      </sensor>
+    </gazebo>
+  </xacro:macro>
 </robot>

File: cp3_base/robot_description/cp3/urdf/turtlebot_properties.urdf.xacro (robot description, xacro)
@@ -19,5 +19,5 @@
      (currently in development and awaiting feedback)
    -->
-	<xacro:property name="cam_px" value="0.25" />
+	<xacro:property name="cam_px" value="0.087" />
 <!--	<xacro:property name="cam_py" value="-0.0125" /> Y varies for different configurations. get sets in sensors_urdf -->
 	<xacro:property name="cam_pz" value="0.2870" />
