Commit message: Moved kinect a bit on robot model to allow collisions

File: cp3_base/robot_description/cp3/urdf/kinect.urdf.xacro (robot description, xacro)
@@ -25,5 +25,5 @@
       <link name="camera_link">
       <visual>
-       <origin xyz="0 0 0" rpy="0 0 ${M_PI/2}"/>
+       <origin xyz="-0.12 0 0" rpy="0 0 ${M_PI/2}"/>
         <geometry>
          <mesh filename="package://turtlebot_description/meshes/sensors/kinect.dae"/>
@@ -31,5 +31,5 @@
       </visual>
   	  <collision>
-        <origin xyz="0.0 0.0 0.0" rpy="0 0 0"/>
+        <origin xyz="-0.12 0.0 0.0" rpy="0 0 0"/>
   	    <geometry>
   	      <box size="0.07271 0.27794 0.073"/>
@@ -38,5 +38,5 @@
       <inertial>
         <mass value="0.564" />
-        <origin xyz="0 0 0" />
+        <origin xyz="-0.12 0 0" />
         <inertia ixx="0.003881243" ixy="0.0" ixz="0.0"
                  iyy="0.000498940" iyz="0.0"

File: cp3_base/robot_description/cp3/urdf/turtlebot_properties.urdf.xacro (robot description, xacro)
@@ -19,5 +19,5 @@
      (currently in development and awaiting feedback)
    -->
-	<xacro:property name="cam_px" value="0.087" />
+	<xacro:property name="cam_px" value="-0.087" />
 <!--	<xacro:property name="cam_py" value="-0.0125" /> Y varies for different configurations. get sets in sensors_urdf -->
 	<xacro:property name="cam_pz" value="0.2870" />
